Commit message: Atlas self-collision works

File: roboschool/models_robot/atlas_description/urdf/atlas_v4_with_multisense.urdf (robot description, URDF)
Before this commit: robot multisense_sl, 31 links, 30 joints
Links:
- link ltorso: geometry visual mesh filename=package://atlas_description/meshes_unplugged/ltorso.dae scale=1 1 1
